Commit message: flip works, connected to odom

File: diff_drive/urdf/ddrive.gazebo.xacro (robot description, xacro)
@@ -8,11 +8,17 @@
             <topic>/cmd_vel</topic>
             <odom_topic>/odom</odom_topic>
+            <tf_topic>/tf</tf_topic>
+            <frame_id>/odom</frame_id>
+            <child_frame_id>/base_link</child_frame_id>
         </plugin>
     </gazebo>
-    <gazebo link="L_front_wheel">
+    <gazebo>
+        <plugin filename="ignition-gazebo-joint-state-publisher-system" name="ignition::gazebo::systems::JointStatePublisher"/>
+    </gazebo>
+    <gazebo Reference="L_front_wheel">
         <mu1>0.2</mu1>
         <mu2>0.2</mu2>
     </gazebo>
-    <gazebo link="R_front_wheel">
+    <gazebo Reference="R_front_wheel">
         <mu1>0.2</mu1>
         <mu2>0.2</mu2>

File: diff_drive/urdf/ddrive.urdf.xacro (robot description, xacro)
@@ -55,5 +55,5 @@
             </geometry>
         </collision>
-        <xacro:box_inertial mass='10' length='${length}' width='${wbody}' height='${hbody}'/>
+        <xacro:box_inertial mass='15' length='${length}' width='${wbody}' height='${hbody}'/>
     </link>
     <xacro:macro name="front_wheels" params="prefix reflect">
@@ -72,10 +72,10 @@
                 </geometry>
                 </collision>
-                <xacro:cyl_inertial mass='5' height='${wwheel}' radius='${rwheel}'/>
+                <xacro:cyl_inertial mass='10' height='${wwheel}' radius='${rwheel}'/>
         </link>
         <joint name="base_to_${prefix}_front_wheel" type="continuous">
             <parent link="base_link"/>
             <child link="${prefix}_front_wheel"/>
-            <origin xyz="${reflect*(wbody/2+wwheel/2)} ${length/2-(rwheel*1.0/3.0)} 0" />
+            <origin xyz="${reflect*(wbody/2+wwheel/2)} ${length/2-(rwheel*1.0/3.0)}  0" />
             <axis xyz="1 0 0"/>
         </joint>
@@ -109,5 +109,5 @@
         <link name="${prefix}_caster_wheel">
             <visual>
-                <origin xyz="0 0 0" rpy="0 ${pi/2}  0" />
+                <origin xyz="0 0 0" rpy="0 ${pi/2} 0" />
                 <geometry>
                     <cylinder radius="${rcaster}" length="0.1" />
@@ -116,10 +116,10 @@
                 </visual>
                 <collision>
-                <origin xyz="0 0 0" rpy="0 ${pi/2}  0"/>
+                <origin xyz="0 0 0" rpy="0 ${pi/2} 0"/>
                 <geometry>
                     <cylinder radius="${rcaster}" length="0.1"/>
                 </geometry>
                 </collision>
-                <xacro:cyl_inertial mass='1' height='${rcaster}' radius='0.1'/>
+                <xacro:cyl_inertial mass='5' height='${rcaster}' radius='0.1'/>
         </link>
         <joint name="base_to_${prefix}_caster_wheel" type="continuous">
